Commit message: make gazebo sim

File: fairino10_v6_moveit2_config/config/fairino10_v6_robot.urdf.xacro (robot description, xacro)
@@ -1,9 +1,19 @@
 <?xml version="1.0"?>
 <robot xmlns:xacro="http://www.ros.org/wiki/xacro" name="fairino10_v6_robot">
+  <link name="world"/>
+  <joint name="world_joint" type="fixed">
+    <origin rpy="0 0 0" xyz="0 0 0"/>
+    <parent link="world"/>
+    <child link="base_link"/>
+  </joint>
     <xacro:arg name="initial_positions_file" default="initial_positions.yaml" />
-    <!-- Import fairino10_v6_robot urdf file -->
+    <!-- Import panda urdf file -->
     <xacro:include filename="$(find fairino_description)/urdf/fairino10_v6.urdf" />
-    <!-- Import control_xacro -->
-    <xacro:include filename="fairino10_v6_robot.ros2_control.xacro" />
+    <!-- Import panda ros2_control description -->
+    <xacro:include filename="fairino10_v6_robot_fake.ros2_control.xacro" />
+    <!-- <xacro:include filename="fairino10_v6_robot_real.ros2_control.xacro" /> -->
+    <!-- <xacro:include filename="fairino10_v6_robot_gazebo.ros2_control.xacro" /> -->
     <xacro:fairino10_v6_robot_ros2_control name="FakeSystem" initial_positions_file="$(arg initial_positions_file)"/>
+    <!-- <xacro:include filename="panda_hand.ros2_control.xacro" /> -->
+    <!-- <xacro:panda_hand_ros2_control name="HandSystem"/> -->
 </robot>

File: fairino_description/urdf/fairino10_v6.urdf (robot description, URDF)
Before this commit: robot fairino10_v6_robot, 8 links, 7 joints
Links:
- removed link world
Joints:
- removed joint world_joint

Commit message: refine moveit simulation

File: fairino10_v6_moveit2_config/config/fairino10_v6_robot.urdf.xacro (robot description, xacro)
@@ -7,13 +7,16 @@
     <child link="base_link"/>
   </joint>
-    <xacro:arg name="initial_positions_file" default="initial_positions.yaml" />
-    <!-- Import panda urdf file -->
-    <xacro:include filename="$(find fairino_description)/urdf/fairino10_v6.urdf" />
-    <!-- Import panda ros2_control description -->
-    <xacro:include filename="fairino10_v6_robot_fake.ros2_control.xacro" />
-    <!-- <xacro:include filename="fairino10_v6_robot_real.ros2_control.xacro" /> -->
-    <!-- <xacro:include filename="fairino10_v6_robot_gazebo.ros2_control.xacro" /> -->
-    <xacro:fairino10_v6_robot_ros2_control name="FakeSystem" initial_positions_file="$(arg initial_positions_file)"/>
-    <!-- <xacro:include filename="panda_hand.ros2_control.xacro" /> -->
-    <!-- <xacro:panda_hand_ros2_control name="HandSystem"/> -->
+  <!-- fake, gazebo, real -->
+  <xacro:arg name="hardware_type" default="fake" />
+  <xacro:arg name="initial_positions_file" default="initial_positions.yaml" />
+  <!-- Your base URDF geometry -->
+  <xacro:include filename="$(find fairino_description)/urdf/fairino10_v6.urdf" />
+  <xacro:include filename="fairino10_v6_robot_fake.ros2_control.xacro" />
+  <xacro:fairino10_v6_robot_ros2_control name="FakeSystem" initial_positions_file="$(arg initial_positions_file)" hardware_type="$(arg hardware_type)"/>
+  <xacro:include filename="fairino10_v6_robot_gazebo.ros2_control.xacro" />
+  <xacro:fairino10_v6_robot_ros2_control name="GazeboSystem" initial_positions_file="$(arg initial_positions_file)" hardware_type="$(arg hardware_type)"/>
+  <xacro:include filename="fairino10_v6_robot_real.ros2_control.xacro" />
+  <xacro:fairino10_v6_robot_ros2_control name="RealSystem" initial_positions_file="$(arg initial_positions_file)" hardware_type="$(arg hardware_type)"/>
+  <!-- <xacro:include filename="panda_hand.ros2_control.xacro" /> -->
+  <!-- <xacro:panda_hand_ros2_control name="HandSystem"/> -->
 </robot>

File: fairino10_v6_moveit2_config/config/fairino10_v6_robot_fake.ros2_control.xacro (robot description, xacro)
@@ -1,5 +1,6 @@
 <?xml version="1.0"?>
 <robot xmlns:xacro="http://www.ros.org/wiki/xacro">
-    <xacro:macro name="fairino10_v6_robot_ros2_control" params="name initial_positions_file">
+    <xacro:macro name="fairino10_v6_robot_ros2_control" params="name initial_positions_file hardware_type">
+      <xacro:if value="${hardware_type == 'fake'}">
         <xacro:property name="initial_positions" value="${xacro.load_yaml(initial_positions_file)['initial_positions']}"/>
         <ros2_control name="${name}" type="system">
@@ -62,4 +63,5 @@
             </joint>
         </ros2_control>
+      </xacro:if>
     </xacro:macro>
 </robot>

File: fairino10_v6_moveit2_config/config/fairino10_v6_robot_gazebo.ros2_control.xacro (robot description, xacro)
@@ -1,5 +1,6 @@
 <?xml version="1.0"?>
 <robot xmlns:xacro="http://www.ros.org/wiki/xacro">
-    <xacro:macro name="fairino10_v6_robot_ros2_control" params="name initial_positions_file">
+    <xacro:macro name="fairino10_v6_robot_ros2_control" params="name initial_positions_file hardware_type">
+      <xacro:if value="${hardware_type == 'gazebo'}">
         <xacro:property name="initial_positions" value="${xacro.load_yaml(initial_positions_file)['initial_positions']}"/>
         <ros2_control name="${name}" type="system">
@@ -62,11 +63,12 @@
             </joint>
         </ros2_control>
+        <gazebo>
+            <plugin filename="libgazebo_ros2_control.so" name="gazebo_ros2_control">
+                <robot_param>robot_description</robot_param>
+                <robot_param_node>robot_state_publisher</robot_param_node>
+                <parameters>/home/vboxuser/colcon_ws/src/frcobot_ros2/fairino10_v6_moveit2_config/config/ros2_controllers.yaml</parameters>
+            </plugin>
+        </gazebo>
+      </xacro:if>
     </xacro:macro>
-    <gazebo>
-        <plugin filename="libgazebo_ros2_control.so" name="gazebo_ros2_control">
-            <robot_param>robot_description</robot_param>
-            <robot_param_node>robot_state_publisher</robot_param_node>
-            <parameters>/home/vboxuser/colcon_ws/src/frcobot_ros2/fairino10_v6_moveit2_config/config/ros2_controllers.yaml</parameters>
-        </plugin>
-    </gazebo>
 </robot>

File: fairino10_v6_moveit2_config/config/fairino10_v6_robot_real.ros2_control.xacro (robot description, xacro)
@@ -1,5 +1,6 @@
 <?xml version="1.0"?>
 <robot xmlns:xacro="http://www.ros.org/wiki/xacro">
-    <xacro:macro name="fairino10_v6_robot_ros2_control" params="name initial_positions_file">
+    <xacro:macro name="fairino10_v6_robot_ros2_control" params="name initial_positions_file hardware_type">
+      <xacro:if value="${hardware_type == 'real'}">
         <xacro:property name="initial_positions" value="${load_yaml(initial_positions_file)['initial_positions']}"/>
         <ros2_control name="${name}" type="system">
@@ -45,4 +46,5 @@
             </joint>
         </ros2_control>
+      </xacro:if>
     </xacro:macro>
 </robot>

Commit message: Fix task_builder task execution errors

File: fairino10_v6_moveit2_config/config/fairino10_v6_robot.urdf.xacro (robot description, xacro)
@@ -1,4 +1,5 @@
 <?xml version="1.0"?>
 <robot xmlns:xacro="http://www.ros.org/wiki/xacro" name="fairino10_v6_robot">
+  <xacro:property name="use_gripper" value="false"/>
   <link name="world"/>
   <joint name="world_joint" type="fixed">
@@ -18,5 +19,21 @@
   <xacro:include filename="fairino10_v6_robot_real.ros2_control.xacro" />
   <xacro:fairino10_v6_robot_ros2_control name="RealSystem" initial_positions_file="$(arg initial_positions_file)" hardware_type="$(arg hardware_type)"/>
-  <!-- <xacro:include filename="panda_hand.ros2_control.xacro" /> -->
-  <!-- <xacro:panda_hand_ros2_control name="HandSystem"/> -->
+  <xacro:if value="${use_gripper}">
+    <link name="tip_link"/>
+    <joint name="tip_joint" type="fixed">
+      <origin rpy="0 0 0.2" xyz="0 0 0"/>
+      <parent link="wrist3_link"/>
+      <child link="tip_link"/>
+    </joint>
+    <!-- <xacro:include filename="panda_hand.ros2_control.xacro" />
+    <xacro:panda_hand_ros2_control name="HandSystem"/> -->
+  </xacro:if>
+  <xacro:unless value="${use_gripper}">
+    <link name="tip_link"/>
+    <joint name="tip_joint" type="fixed">
+      <origin rpy="0 0 0" xyz="0 0 0.2"/>
+      <parent link="wrist3_link"/>
+      <child link="tip_link"/>
+    </joint>
+  </xacro:unless>
 </robot>

Commit message: Fix executor and add depth sensor pipeline

File: fairino10_v6_moveit2_config/config/fairino10_v6_robot.urdf.xacro (robot description, xacro)
@@ -13,4 +13,60 @@
   <!-- Your base URDF geometry -->
   <xacro:include filename="$(find fairino_description)/urdf/fairino10_v6.urdf" />
+  <!-- Conditionally add depth camera if using gazebo -->
+    <!-- Depth Camera Link -->
+    <link name="camera_link">
+      <visual>
+        <origin xyz="0 0 0" rpy="0 0 0"/>
+        <geometry>
+          <box size="0.1 0.1 0.1"/>
+        </geometry>
+        <material name="gray">
+          <color rgba="0.5 0.5 0.5 1"/>
+        </material>
+      </visual>
+      <collision>
+        <origin xyz="0 0 0" rpy="0 0 0"/>
+        <geometry>
+          <box size="0.1 0.1 0.1"/>
+        </geometry>
+      </collision>
+    </link>
+    <!-- Depth Camera Joint (attach camera_link to base_link) -->
+    <joint name="camera_joint" type="fixed">
+      <origin xyz="0.2 0 0.8" rpy="0 0 0"/>
+      <parent link="base_link"/>
+      <child link="camera_link"/>
+    </joint>
+    <!-- Gazebo sensor plugin for depth simulation -->
+    <gazebo reference="camera_link">
+      <sensor type="depth" name="depth_sensor">
+        <update_rate>30</update_rate>
+        <camera>
+          <horizontal_fov>1.047</horizontal_fov>
+          <image>
+            <width>640</width>
+            <height>480</height>
+          </image>
+          <clip>
+            <near>0.1</near>
+            <far>5.0</far>
+          </clip>
+        </camera>
+        <plugin name="camera_driver1" filename="libgazebo_ros_camera.so">
+            <!-- Keep plugin at 30 Hz -->
+            <update_rate>30</update_rate>
+            <camera_name>camera_depth</camera_name>
+            <frame_name>camera_depth</frame_name>
+            <!-- Topics as requested -->
+            <imageTopicName>/camera_depth/image_raw</imageTopicName>
+            <cameraInfoTopicName>/camera_depth/camera_info</cameraInfoTopicName>
+            <depthImageTopicName>/camera_depth/depth/image_raw</depthImageTopicName>
+            <!-- Approximate OAK-D Lite stereo baseline of ~7.5 cm -->
+            <hack_baseline>0.075</hack_baseline>
+            <min_depth>0.2</min_depth>
+            <max_depth>9.0</max_depth>
+        </plugin>
+      </sensor>
+    </gazebo>
   <xacro:include filename="fairino10_v6_robot_fake.ros2_control.xacro" />
   <xacro:fairino10_v6_robot_ros2_control name="FakeSystem" initial_positions_file="$(arg initial_positions_file)" hardware_type="$(arg hardware_type)"/>

Commit message: Fix depth sensor pipeline

File: fairino10_v6_moveit2_config/config/fairino10_v6_robot.urdf.xacro (robot description, xacro)
@@ -34,5 +34,5 @@
     <!-- Depth Camera Joint (attach camera_link to base_link) -->
     <joint name="camera_joint" type="fixed">
-      <origin xyz="0.2 0 0.8" rpy="0 0 0"/>
+      <origin xyz="0.2 0 0.8" rpy="0 0.2 0"/>
       <parent link="base_link"/>
       <child link="camera_link"/>
@@ -41,5 +41,5 @@
     <gazebo reference="camera_link">
       <sensor type="depth" name="depth_sensor">
-        <update_rate>30</update_rate>
+        <update_rate>10</update_rate>
         <camera>
           <horizontal_fov>1.047</horizontal_fov>
@@ -54,8 +54,8 @@
         </camera>
         <plugin name="camera_driver1" filename="libgazebo_ros_camera.so">
-            <!-- Keep plugin at 30 Hz -->
-            <update_rate>30</update_rate>
+            <!-- Keep plugin at 10 Hz -->
+            <update_rate>20</update_rate>
             <camera_name>camera_depth</camera_name>
-            <frame_name>camera_depth</frame_name>
+            <frame_name>camera_link</frame_name>
             <!-- Topics as requested -->
             <imageTopicName>/camera_depth/image_raw</imageTopicName>

Commit message: Fix the the depth sensor pipeline

File: fairino10_v6_moveit2_config/config/fairino10_v6_robot.urdf.xacro (robot description, xacro)
@@ -34,7 +34,20 @@
     <!-- Depth Camera Joint (attach camera_link to base_link) -->
     <joint name="camera_joint" type="fixed">
-      <origin xyz="0.2 0 0.8" rpy="0 0.2 0"/>
+      <origin xyz="0.6 0 0.8" rpy="0 0.2 3.14"/>
       <parent link="base_link"/>
       <child link="camera_link"/>
+    </joint>
+    <link name="camera_phantom_link">
+        <origin xyz="0 0 0" rpy="0 0 0"/>
+        <inertial>
+            <origin xyz="0 0 0" rpy="0 0 0" />
+            <mass value="0.001" />
+            <inertia ixx="0.0001" ixy="9.9865E-08" ixz="7.787E-08" iyy="0.0001" iyz="6.6716E-08" izz="0.0001" />
+        </inertial>
+    </link>
+    <joint name="camera_phantom_joint" type="fixed">
+        <parent link="camera_link"/>
+        <child link="camera_phantom_link"/>
+        <origin xyz="0 0 0" rpy="-1.57 0 -1.57"/>
     </joint>
     <!-- Gazebo sensor plugin for depth simulation -->
@@ -57,5 +70,5 @@
             <update_rate>20</update_rate>
             <camera_name>camera_depth</camera_name>
-            <frame_name>camera_link</frame_name>
+            <frame_name>camera_phantom_link</frame_name>
             <!-- Topics as requested -->
             <imageTopicName>/camera_depth/image_raw</imageTopicName>

Commit message: Fix sensor pipeline and add gripper_description

File: fairino10_v6_moveit2_config/config/fairino10_v6_robot.urdf.xacro (robot description, xacro)
@@ -11,75 +11,8 @@
   <xacro:arg name="hardware_type" default="fake" />
   <xacro:arg name="initial_positions_file" default="initial_positions.yaml" />
-  <!-- Your base URDF geometry -->
+  <!-- Camera URDF -->
+  <xacro:include filename="$(find depth_camera_description)/urdf/depth_camera.urdf" />
+  <!-- Robot base URDF -->
   <xacro:include filename="$(find fairino_description)/urdf/fairino10_v6.urdf" />
-  <!-- Conditionally add depth camera if using gazebo -->
-    <!-- Depth Camera Link -->
-    <link name="camera_link">
-      <visual>
-        <origin xyz="0 0 0" rpy="0 0 0"/>
-        <geometry>
-          <box size="0.1 0.1 0.1"/>
-        </geometry>
-        <material name="gray">
-          <color rgba="0.5 0.5 0.5 1"/>
-        </material>
-      </visual>
-      <collision>
-        <origin xyz="0 0 0" rpy="0 0 0"/>
-        <geometry>
-          <box size="0.1 0.1 0.1"/>
-        </geometry>
-      </collision>
-    </link>
-    <!-- Depth Camera Joint (attach camera_link to base_link) -->
-    <joint name="camera_joint" type="fixed">
-      <origin xyz="0.6 0 0.8" rpy="0 0.2 3.14"/>
-      <parent link="base_link"/>
-      <child link="camera_link"/>
-    </joint>
-    <link name="camera_phantom_link">
-        <origin xyz="0 0 0" rpy="0 0 0"/>
-        <inertial>
-            <origin xyz="0 0 0" rpy="0 0 0" />
-            <mass value="0.001" />
-            <inertia ixx="0.0001" ixy="9.9865E-08" ixz="7.787E-08" iyy="0.0001" iyz="6.6716E-08" izz="0.0001" />
-        </inertial>
-    </link>
-    <joint name="camera_phantom_joint" type="fixed">
-        <parent link="camera_link"/>
-        <child link="camera_phantom_link"/>
-        <origin xyz="0 0 0" rpy="-1.57 0 -1.57"/>
-    </joint>
-    <!-- Gazebo sensor plugin for depth simulation -->
-    <gazebo reference="camera_link">
-      <sensor type="depth" name="depth_sensor">
-        <update_rate>10</update_rate>
-        <camera>
-          <horizontal_fov>1.047</horizontal_fov>
-          <image>
-            <width>640</width>
-            <height>480</height>
-          </image>
-          <clip>
-            <near>0.1</near>
-            <far>5.0</far>
-          </clip>
-        </camera>
-        <plugin name="camera_driver1" filename="libgazebo_ros_camera.so">
-            <!-- Keep plugin at 10 Hz -->
-            <update_rate>20</update_rate>
-            <camera_name>camera_depth</camera_name>
-            <frame_name>camera_phantom_link</frame_name>
-            <!-- Topics as requested -->
-            <imageTopicName>/camera_depth/image_raw</imageTopicName>
-            <cameraInfoTopicName>/camera_depth/camera_info</cameraInfoTopicName>
-            <depthImageTopicName>/camera_depth/depth/image_raw</depthImageTopicName>
-            <!-- Approximate OAK-D Lite stereo baseline of ~7.5 cm -->
-            <hack_baseline>0.075</hack_baseline>
-            <min_depth>0.2</min_depth>
-            <max_depth>9.0</max_depth>
-        </plugin>
-      </sensor>
-    </gazebo>
   <xacro:include filename="fairino10_v6_robot_fake.ros2_control.xacro" />
   <xacro:fairino10_v6_robot_ros2_control name="FakeSystem" initial_positions_file="$(arg initial_positions_file)" hardware_type="$(arg hardware_type)"/>

Commit message: Add gripper hardware package

File: fairino10_v6_moveit2_config/config/fairino10_v6_robot.urdf.xacro (robot description, xacro)
@@ -1,5 +1,5 @@
 <?xml version="1.0"?>
 <robot xmlns:xacro="http://www.ros.org/wiki/xacro" name="fairino10_v6_robot">
-  <xacro:property name="use_gripper" value="false"/>
+  <xacro:property name="use_gripper" value="true"/>
   <link name="world"/>
   <joint name="world_joint" type="fixed">
@@ -28,6 +28,11 @@
       <child link="tip_link"/>
     </joint>
-    <!-- <xacro:include filename="panda_hand.ros2_control.xacro" />
-    <xacro:panda_hand_ros2_control name="HandSystem"/> -->
+    <xacro:include filename="$(find fairino_description)/urdf/gripper.urdf" />
+    <!-- <xacro:include filename="gripper.ros2_control.xacro" />
+    <xacro:gripper_ros2_control name="FakeSystem" initial_positions_file="$(arg initial_positions_file)" hardware_type="$(arg hardware_type)"/>
+    <xacro:include filename="gripper.ros2_control.xacro" />
+    <xacro:gripper_ros2_control name="GazeboSystem" initial_positions_file="$(arg initial_positions_file)" hardware_type="$(arg hardware_type)"/>
+    <xacro:include filename="gripper.ros2_control.xacro" />
+    <xacro:gripper_ros2_control name="RealSystem" initial_positions_file="$(arg initial_positions_file)" hardware_type="$(arg hardware_type)"/> -->
   </xacro:if>
   <xacro:unless value="${use_gripper}">

File: fairino_description/urdf/gripper.urdf (robot description, URDF)
Before this commit: robot gripper, 4 links, 3 joints
Links:
- link hand_hand: geometry collision cylinder length=0.1 radius=0.02; collision cylinder length=0.1 radius=0.04
- link hand_leftfinger: geometry visual mesh filename=package://fairino_description/meshes/gripper/finger.dae
- link hand_rightfinger: geometry visual mesh filename=package://fairino_description/meshes/gripper/finger.dae
Joints:
- added joint base_joint: type fixed, parent wrist3_link, child hand_hand, origin xyz=0.0 0.0 0.1134 rpy=0 0 1.57

Commit message: Port hardware V3.0

File: fairino10_v6_moveit2_config/config/fairino10_v6_robot.urdf.xacro (robot description, xacro)
@@ -1,5 +1,6 @@
 <?xml version="1.0"?>
 <robot xmlns:xacro="http://www.ros.org/wiki/xacro" name="fairino10_v6_robot">
-  <xacro:property name="use_gripper" value="true"/>
+  <xacro:property name="use_gripper" value="false"/>
+  <xacro:property name="use_sensor" value="false"/>
   <link name="world"/>
   <joint name="world_joint" type="fixed">
@@ -9,8 +10,10 @@
   </joint>
   <!-- fake, gazebo, real -->
-  <xacro:arg name="hardware_type" default="fake" />
+  <xacro:arg name="hardware_type" default="real" />
   <xacro:arg name="initial_positions_file" default="initial_positions.yaml" />
   <!-- Camera URDF -->
-  <xacro:include filename="$(find depth_camera_description)/urdf/depth_camera.urdf" />
+  <xacro:if value="${use_sensor}">
+    <xacro:include filename="$(find depth_camera_description)/urdf/depth_camera.urdf" />
+  </xacro:unless>
   <!-- Robot base URDF -->
   <xacro:include filename="$(find fairino_description)/urdf/fairino10_v6.urdf" />

File: fairino10_v6_moveit2_config/config/fairino10_v6_robot_real.ros2_control.xacro (robot description, xacro)
@@ -6,6 +6,9 @@
         <ros2_control name="${name}" type="system">
             <hardware>
-                <!-- By default, set up controllers for simulation. This won't work on real hardware -->
-                <plugin>mock_components/GenericSystem</plugin>
+                <!--
+                Modify the CONTROLLER_IP in fairino_hardware\data_type_def.h from the default value "192.168.58.2" to the actual robot's IP address.
+                Modify the CONTROLLER_IP_ADDRESS in fairino_hardware\include\fairino_hardware\fairino_hardware_interface.hpp from the default value "192.168.58.2" to the actual robot's IP address.
+                -->
+                <plugin>fairino_hardware/FairinoHardwareInterface</plugin>
             </hardware>
             <joint name="j1">
